Commit message: feat: add MuJoCo pick-place V4 simulation validation

File: src/drok_arm_description/urdf/drok_arm.urdf (robot description, URDF)
Before this commit: robot DROK_P_gripper_D405, 12 links, 11 joints
Links:
- link GRIPPER_BASE: geometry visual mesh filename=package://drok_arm_description/meshes/GRIPPER_BASE.STL
- link GRIPPER_LEFT: geometry collision box size=0.040 0.003 0.040; visual box size=0.040 0.003 0.040
- link GRIPPER_RIGH: geometry collision box size=0.040 0.003 0.040; visual box size=0.040 0.003 0.040

File: src/drok_arm_mujoco/urdf/drok_arm_mujoco.urdf (robot description, URDF)
Before this commit: robot DROK_P_gripper_D405, 12 links, 11 joints
Links:
- link GRIPPER_BASE: geometry visual mesh filename=package://drok_arm_description/meshes/GRIPPER_BASE.STL
- link GRIPPER_LEFT: geometry collision box size=0.040 0.003 0.040; visual mesh filename=package://drok_arm_description/meshes/GRIPPER_LEFT.STL
- link GRIPPER_RIGH: geometry collision box size=0.040 0.003 0.040; visual mesh filename=package://drok_arm_description/meshes/GRIPPER_RIGH.STL
Joints:
- joint GRIPPER_RIGHT_JOINT: axis (none) -> 0 -1 0; limit (none) -> lower=-0.04 upper=0.0 effort=100.0 velocity=0.05; type fixed -> prismatic
- joint JOINT7: axis (none) -> 0 -1 0; limit (none) -> lower=0.0 upper=0.04 effort=100.0 velocity=0.05; type fixed -> prismatic
