Commit message: feat: Pick and Place 1 Way

File: src/drok_arm_mujoco/urdf/drok_arm_mujoco.urdf (robot description, URDF)
Before this commit: robot DROK_P_gripper_D405, 12 links, 11 joints
Joints:
- joint GRIPPER_RIGHT_JOINT: limit lower=-0.04 upper=0.0 effort=100.0 velocity=0.05 -> lower=-0.05 upper=0.0 effort=100.0 velocity=0.05
- joint JOINT7: limit lower=0.0 upper=0.04 effort=100.0 velocity=0.05 -> lower=0.0 upper=0.05 effort=100.0 velocity=0.05

Commit message: feat: add stateful multi-box pick and place

File: src/drok_arm_mujoco/urdf/drok_arm_mujoco.urdf (robot description, URDF)
Before this commit: robot DROK_P_gripper_D405, 12 links, 11 joints
Joints:
- joint JOINT1: limit lower=-0.78540 upper=2.26893 effort=35 velocity=1.2 -> lower=-6.50000 upper=6.50000 effort=35 velocity=1.2
